File: random ass keyboard.kicad_sch (KiCad schematic)
At the start: 78 parts, among them J1 USB_C, SW1 SW_Push, U1 STM32F072CBT6, U3 XC6206, U4 USBLC6-2SC6

Commit message: schem
Parts:
- removed D45: Diode, ScottoKeebs_Components:Diode_SOD-123, symbol ScottoKeebs:Placeholder_Diode
- removed MT1: PEC11R-4215F-S0024, ec11:RotaryEncoder_Alps_EC11E-Switch_Vertical_H20mm, symbol ec11:PEC11R-4215F-S0024
- added D34: Diode, ScottoKeebs_Components:Diode_SOD-123, symbol ScottoKeebs:Placeholder_Diode
- added SW2: RotaryEncoder_Switch, Rotary_Encoder:RotaryEncoder_Alps_EC11E-Switch_Vertical_H20mm_CircularMountingHoles, symbol Device:RotaryEncoder_Switch
Connections:
- net B0: now also SW2.A
- net B1: now also SW2.B
- net GND: now also SW2.C
- net col0: now also SW2.S1
- net row4: now also D34.1 (K)
- new net: D34.2 (A), SW2.S2

Commit message: i... actually finished this shit.
Connections:
- net A3 is gone; now on net row0: U1.13 (PA3)
- net A4 is gone; now on net row1: U1.14 (PA4)
- net A5 is gone; now on net row2: U1.15 (PA5)
- net A6 is gone; now on net row3: U1.16 (PA6)
- net A10: no longer U1.31 (PA10)
- net B0: now also SW2.B; no longer SW2.A
- net B1: now also SW2.A; no longer SW2.B
- net col0: now also U1.22 (PB11); no longer U1.20 (PB2)
- net col1: now also U1.42 (PB6); no longer U1.39 (PB3)
- net col2: now also U1.43 (PB7); no longer U1.40 (PB4)
- net col3: now also U1.45 (PB8); no longer U1.41 (PB5)
- net col4: now also U1.46 (PB9); no longer U1.42 (PB6)
- net row0: no longer U1.43 (PB7)
- net row1: no longer U1.45 (PB8)
- net row2: no longer U1.46 (PB9)
- net row3: no longer U1.21 (PB10)
- net row4: now also U1.31 (PA10); no longer U1.22 (PB11)
- net at D28.2 (DOUT): now also D8.4 (DIN)
- net at D30.4 (DIN): now also R4.2; no longer D31.2 (DOUT)
- net A7: no longer names the net of U1.17 (PA7)
- new net B10: U1.21 (PB10)
- new net B2: U1.20 (PB2)
- new net B3: U1.39 (PB3)
- new net B4: U1.40 (PB4)
- new net B5: U1.41 (PB5)
Other:
- moved on the sheet: R4

Commit message: other things
Parts:
- SW2: footprint Rotary_Encoder:RotaryEncoder_Alps_EC11E-Switch_Vertical_H20mm_CircularMountingHoles -> Rotary_Encoder:RotaryEncoder_Alps_EC11E-Switch_Vertical_H20mm_MountingHoles
Changed lines of the file:
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@@
 			)
 		)
-		(property "Footprint" "Rotary_Encoder:RotaryEncoder_Alps_EC11E-Switch_Vertical_H20mm_CircularMountingHoles"
+		(property "Footprint" "Rotary_Encoder:RotaryEncoder_Alps_EC11E-Switch_Vertical_H20mm_MountingHoles"
 			(at 162.56 79.756 0)
 			(effects

Commit message: updated that one diode
Parts:
- D23: LCSC (none) -> C2128
